File: docs/schematics/reference-project/reference-project.kicad_pcb (KiCad board)
At the start: 2 copper layers, 22 parts, among them J1 UART, Q1 MMBT3904, SW1 INPUT_0, SW2 INPUT_1, SW3 INPUT_2, SW4 INPUT_3, SW5 INPUT_4, SW6 INPUT_5, SW7 RESET, U1 74HC165D, U2 ATTINY85-20PU

Commit message: Finished schematics.
Parts:
- added BT1: CELL, Connectors:bornier2, F.Cu at (53.1, 62.7)
- moved R7 122.3 mm to (52.7, 69.5)
- moved U2 119.5 mm to (57.9, 73.8), turned to 270 degrees
- moved R9 108.8 mm to (62.0, 66.5), turned to 0 degrees
- moved Q1 107.8 mm to (57.9, 69.8), turned to 90 degrees
- moved R8 106.2 mm to (63.8, 74.3), turned to 180 degrees
- moved SW1 104.3 mm to (63.8, 112.8)
- moved SW5 103.7 mm to (55.3, 112.8)
- moved D1 102.8 mm to (63.4, 70.3), turned to 90 degrees
- moved R4 102.8 mm to (60.2, 96.7), turned to 270 degrees
- moved J1 101.2 mm to (59.2, 62.6), turned to 0 degrees
- moved R2 101.0 mm to (65.0, 97.4), turned to 270 degrees
- moved R1 98.2 mm to (67.3, 96.7), turned to 270 degrees
- moved U1 97.1 mm to (63.7, 87.9)
- moved LS1 95.8 mm to (68.8, 73.1), turned to 0 degrees
- moved SW4 95.7 mm to (72.4, 106.3), turned to 180 degrees
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Connections:
- U2 pad 5: Net-(U1-Pad9) -> Net-(U1-Pad7)
Routing:
- net +3V3: track 0.00 -> 176.4 mm
- net Net-(R7-Pad2): track 0.00 -> 69.9 mm
- net Net-(R3-Pad1): track 0.00 -> 42.3 mm
- net Net-(R5-Pad1): track 0.00 -> 39.4 mm
- net Net-(R4-Pad1): track 0.00 -> 36.1 mm
- net Net-(R1-Pad1): track 0.00 -> 32.3 mm
- net Net-(R6-Pad1): track 0.00 -> 29.1 mm
- net Net-(R2-Pad1): track 0.00 -> 28.4 mm
- net Net-(U1-Pad2): track 0.00 -> 28.1 mm, vias 0 -> 2
- net Net-(U1-Pad7): track 0.00 -> 21.2 mm, vias 0 -> 2
- net Net-(D1-Pad1): track 0.00 -> 19.2 mm
- net Net-(D1-Pad3): track 0.00 -> 8.87 mm
- net Net-(Q1-Pad1): track 0.00 -> 6.96 mm
- net Net-(U1-Pad1): track 0.00 -> 6.75 mm
- net Net-(J1-Pad2): track 0.00 -> 6.28 mm
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- added copper zone on F.Cu, net GND
Other:
- board outline added: 38 x 68 mm
- net class Default: clearance 0.2 -> 0.3; trace_width 0.25 -> 0.381; via_dia 0.6 -> 1.5; via_drill 0.4 -> 0.9
- rule trace_clearance: 0.2 -> 0.3
- rule trace_min: 0.2 -> 0.254
- rule via_min_drill: 0.3 -> 0.9
- rule via_min_size: 0.4 -> 1.5
