File: stm32-f0-rust/docs/schematics/blocks/stm32/stm32.sch (KiCad schematic (older format))
At the start: 3 parts, among them J1 Conn_01x05_Female, J2 Conn_01x02_Female, U1 STM32F042F4Px

Commit message: [PCB][STM32-Block] Use correct footprints for the pin sockets.
Parts:
- J1: footprint (none) -> Connector_PinSocket_2.54mm:PinSocket_1x05_P2.54mm_Vertical
- J2: footprint (none) -> Connector_PinSocket_2.54mm:PinSocket_1x02_P2.54mm_Vertical
Changed lines of the file:
@@
 EESchema Schematic File Version 4
+LIBS:stm32-cache
 EELAYER 26 0
 EELAYER END
@@
 F 0 "J1" H 10327 1576 50  0000 L CNN
 F 1 "Conn_01x05_Female" H 10327 1485 50  0000 L CNN
-F 2 "" H 10300 1550 50  0001 C CNN
+F 2 "Connector_PinSocket_2.54mm:PinSocket_1x05_P2.54mm_Vertical" H 10300 1550 50  0001 C CNN
 F 3 "~" H 10300 1550 50  0001 C CNN
 	1    10300 1550
@@
 F 0 "J2" H 10327 2076 50  0000 L CNN
 F 1 "Conn_01x02_Female" H 10327 1985 50  0000 L CNN
-F 2 "" H 10300 2100 50  0001 C CNN
+F 2 "Connector_PinSocket_2.54mm:PinSocket_1x02_P2.54mm_Vertical" H 10300 2100 50  0001 C CNN
 F 3 "~" H 10300 2100 50  0001 C CNN
 	1    10300 2100

Commit message: [PCB][STM32-Block] Use single 7-pin socket instead of two.
Parts:
- removed J1: Conn_01x05_Female, Connector_PinSocket_2.54mm:PinSocket_1x05_P2.54mm_Vertical, symbol Connector_Generic:Conn_01x05_Female
- removed J2: Conn_01x02_Female, Connector_PinSocket_2.54mm:PinSocket_1x02_P2.54mm_Vertical, symbol Connector_Generic:Conn_01x02_Female
- added J1: Conn_01x07_Female, Connector_PinSocket_2.54mm:PinSocket_1x07_P2.54mm_Horizontal, symbol Connector_Generic:Conn_01x07_Female
Changed lines of the file:
@@
 Comment4 ""
 $EndDescr
-$Comp
-L Connector_Generic:Conn_01x05_Female J1
-U 1 1 5AE8B0F8
-P 10300 1550
-F 0 "J1" H 10327 1576 50  0000 L CNN
-F 1 "Conn_01x05_Female" H 10327 1485 50  0000 L CNN
-F 2 "Connector_PinSocket_2.54mm:PinSocket_1x05_P2.54mm_Vertical" H 10300 1550 50  0001 C CNN
-F 3 "~" H 10300 1550 50  0001 C CNN
-	1    10300 1550
-	1    0    0    -1
-$EndComp
-$Comp
-L Connector_Generic:Conn_01x02_Female J2
-U 1 1 5AE8B17F
-P 10300 2100
-F 0 "J2" H 10327 2076 50  0000 L CNN
-F 1 "Conn_01x02_Female" H 10327 1985 50  0000 L CNN
-F 2 "Connector_PinSocket_2.54mm:PinSocket_1x02_P2.54mm_Vertical" H 10300 2100 50  0001 C CNN
-F 3 "~" H 10300 2100 50  0001 C CNN
-	1    10300 2100
-	1    0    0    -1
-$EndComp
-Text GLabel 10100 1450 0    50   Input ~ 0
+Text GLabel 9100 1700 0    50   Input ~ 0
 SWCLK
-Text GLabel 10100 1650 0    50   Input ~ 0
+Text GLabel 9100 1600 0    50   Input ~ 0
 SWDIO
-Text GLabel 10100 1750 0    50   Input ~ 0
+Text GLabel 9100 1800 0    50   Input ~ 0
 NRST
-Text GLabel 10100 2100 0    50   Input ~ 0
+Text GLabel 9100 1200 0    50   Input ~ 0
 Button
-Text GLabel 10100 2200 0    50   Input ~ 0
+Text GLabel 9100 1300 0    50   Input ~ 0
 Buzzer
 Text GLabel 2800 2550 0    50   Input ~ 0
@@
 	0    1    1    0
 $EndComp
-Text GLabel 10100 1550 0    50   Input ~ 0
+Text GLabel 9100 1400 0    50   Input ~ 0
 GND
 Wire Wire Line
@@
 	0    1    1    0
 $EndComp
-Text GLabel 10100 1350 0    50   Input ~ 0
+Text GLabel 9100 1500 0    50   Input ~ 0
 VDD
+$Comp
+L Connector_Generic:Conn_01x07_Female J1
+U 1 1 5AE8B9BA
+P 9300 1500
+F 0 "J1" H 9327 1526 50  0000 L CNN
+F 1 "Conn_01x07_Female" H 9327 1435 50  0000 L CNN
+F 2 "Connector_PinSocket_2.54mm:PinSocket_1x07_P2.54mm_Horizontal" H 9300 1500 50  0001 C CNN
+F 3 "~" H 9300 1500 50  0001 C CNN
+	1    9300 1500
+	1    0    0    -1
+$EndComp
 $EndSCHEMATC

Commit message: Add correct footprint for smt32 TSSOP-20.
Parts:
- U1: footprint Package_SO:TSSOP-20_4.4x6.5mm_P0.65mm -> digikey-footprints:TSSOP-20_W4.4mm
Changed lines of the file:
@@
 F 0 "U1" H 4650 3400 50  0000 C CNN
 F 1 "STM32F042F4Px" H 5700 1900 50  0000 C CNN
-F 2 "Package_SO:TSSOP-20_4.4x6.5mm_P0.65mm" H 8500 4025 50  0001 R TNN
+F 2 "digikey-footprints:TSSOP-20_W4.4mm" H 8500 4025 50  0001 R TNN
 F 3 "http://www.st.com/st-web-ui/static/active/en/resource/technical/document/datasheet/DM00105814.pdf" H 5700 3150 50  0001 C CNN
 	1    5700 3150
