File: avr-attiny85/docs/schematics/reference-project/reference-project.sch (KiCad schematic (older format))
At the start: 7 parts, among them J1 Conn_01x08_Female, SW1 RESET, SW2 INPUT_5, U1 ATTINY85-20SU

Commit message: Update dependencies + re-generate proxies with the latest svd2rust.
Parts:
- J1: symbol Conn_01x08_Female -> reference-project-rescue:Conn_01x08_Female
- R1, R2, R3: symbol R -> reference-project-rescue:R
- SW1, SW2: symbol SW_Push -> Switch:SW_Push
- U1: symbol ATTINY85-20SU -> reference-project-rescue:ATTINY85-20SU
Changed lines of the file:
@@
-EESchema Schematic File Version 3
-LIBS:power
-LIBS:device
-LIBS:linear
-LIBS:regul
-LIBS:adc-dac
-LIBS:memory
-LIBS:xilinx
-LIBS:microcontrollers
-LIBS:dsp
-LIBS:microchip
-LIBS:analog_switches
-LIBS:motorola
-LIBS:texas
-LIBS:intel
-LIBS:audio
-LIBS:interface
-LIBS:digital-audio
-LIBS:philips
-LIBS:cypress
-LIBS:siliconi
-LIBS:opto
-LIBS:atmel
-LIBS:contrib
-LIBS:User-Submitted
-LIBS:Teensy_3_and_LC_Series_Boards_v1.1
-LIBS:SparkFun-Sensors
-LIBS:SparkFun-Resistors
-LIBS:SparkFun-RF
-LIBS:SparkFun-PowerIC
-LIBS:SparkFun-Passives
-LIBS:SparkFun-LED
-LIBS:SparkFun-FreqCtrl
-LIBS:SparkFun-Electromechanical
-LIBS:SparkFun-DiscreteSemi
-LIBS:SparkFun-DigitalIC
-LIBS:SparkFun-Connectors
-LIBS:SparkFun-Capacitors
-LIBS:SparkFun-Boards
-LIBS:SparkFun-AnalogIC
-LIBS:SparkFun-Aesthetics
-LIBS:LilyPad-Wearables
-LIBS:GeekAmmo
-LIBS:Switch
-LIBS:Relay
-LIBS:Motor
-LIBS:Connector
-LIBS:Transistor
-LIBS:Display
-LIBS:Valve
-LIBS:Logic_74xgxx
-LIBS:Logic_74xx
-LIBS:Logic_CMOS_4000
-LIBS:Logic_CMOS_IEEE
-LIBS:reference-project
-LIBS:Abracon
-LIBS:ActiveSemi
-LIBS:Altera
-LIBS:AMS
-LIBS:AnalogDevices
-LIBS:AOS
-LIBS:Atmel
-LIBS:Bosch
-LIBS:conn-2mm
-LIBS:conn-100mil
-LIBS:conn-amphenol
-LIBS:conn-assmann
-LIBS:conn-cui
-LIBS:conn-fci
-LIBS:conn-jae
-LIBS:conn-linx
-LIBS:conn-molex
-LIBS:conn-special-headers
-LIBS:conn-tagconnect
-LIBS:conn-te
-LIBS:conn-test
-LIBS:DiodesInc
-LIBS:display
-LIBS:electomech-misc
-LIBS:_electromech
-LIBS:Fairchild
-LIBS:FTDI
-LIBS:Infineon
-LIBS:Intersil
-LIBS:Lattice
-LIBS:_linear
-LIBS:LinearTech
-LIBS:Littelfuse
-LIBS:_logic
-LIBS:logic-4000
-LIBS:logic-7400
-LIBS:logic-7400-new
-LIBS:MACOM
-LIBS:Macrofab
-LIBS:maxim
-LIBS:mechanical
-LIBS:Microchip
-LIBS:Micron
-LIBS:Murata
-LIBS:NXP
-LIBS:OceanOptics
-LIBS:onsemi
-LIBS:_passive
-LIBS:pasv-BelFuse
-LIBS:pasv-BiTech
-LIBS:pasv-Bourns
-LIBS:pasv-cap
-LIBS:pasv-ind
-LIBS:pasv-Murata
-LIBS:pasv-res
-LIBS:pasv-TDK
-LIBS:pasv-xtal
-LIBS:pcb
-LIBS:Recom
-LIBS:Richtek
-LIBS:_semi
-LIBS:semi-diode-DiodesInc
-LIBS:semi-diode-generic
-LIBS:semi-diode-MCC
-LIBS:semi-diode-NXP
-LIBS:semi-diode-OnSemi
-LIBS:semi-diode-Semtech
-LIBS:semi-diode-ST
-LIBS:semi-diode-Toshiba
-LIBS:semi-opto-generic
-LIBS:semi-opto-liteon
-LIBS:semi-thyristor-generic
-LIBS:semi-trans-AOS
-LIBS:semi-trans-DiodesInc
-LIBS:semi-trans-EPC
-LIBS:semi-trans-Fairchild
-LIBS:semi-trans-generic
-LIBS:semi-trans-Infineon
-LIBS:semi-trans-IRF
-LIBS:semi-trans-IXYS
-LIBS:semi-trans-NXP
-LIBS:semi-trans-OnSemi
-LIBS:semi-trans-Panasonic
-LIBS:semi-trans-ST
-LIBS:semi-trans-TI
-LIBS:semi-trans-Toshiba
-LIBS:semi-trans-Vishay
-LIBS:silabs
-LIBS:skyworks
-LIBS:ST
-LIBS:st_ic
-LIBS:supertex
-LIBS:symbol
-LIBS:TexasInstruments
-LIBS:u-blox
-LIBS:Vishay
-LIBS:Winbond
-LIBS:Xilinx
+EESchema Schematic File Version 4
 LIBS:reference-project-cache
 EELAYER 26 0
@@
 $EndDescr
 $Comp
-L SW_Push SW1
+L Switch:SW_Push SW1
 U 1 1 59E49B79
 P 9150 5300
@@
 $EndComp
 $Comp
-L SW_Push SW2
+L Switch:SW_Push SW2
 U 1 1 59E49BEA
 P 9800 5300
@@
 $EndComp
 $Comp
-L R R2
+L reference-project-rescue:R R2
 U 1 1 59E53A35
 P 8850 4650
@@
 $EndComp
 $Comp
-L R R3
+L reference-project-rescue:R R3
 U 1 1 59E56D49
 P 9800 4000
@@
 $EndComp
 $Comp
-L R R1
+L reference-project-rescue:R R1
 U 1 1 59E587BF
 P 8850 3600
@@
 $EndComp
 $Comp
-L PWR_FLAG #FLG01
+L power:PWR_FLAG #FLG01
 U 1 1 59E6375F
 P 7850 2250
@@
 $EndComp
 $Comp
-L ATTINY85-20SU U1
+L reference-project-rescue:ATTINY85-20SU U1
 U 1 1 59FA3237
 P 7400 4150
@@
 $EndComp
 $Comp
-L Conn_01x08_Female J1
+L reference-project-rescue:Conn_01x08_Female J1
 U 1 1 59FCBF1A
 P 9100 1850
@@
 	9950 4000 10350 4000
 Wire Wire Line
-	8750 4000 9650 4000
-Wire Wire Line
-	8750 4200 9350 4200
+	8750 4000 9250 4000
+Wire Wire Line
+	8750 4200 8850 4200
 Wire Wire Line
 	8850 4200 8850 3750
@@
 	6050 3000 6050 3900
 Wire Wire Line
-	8750 4300 9600 4300
+	8750 4300 8850 4300
 Wire Wire Line
 	8850 4300 8850 4500
@@
 	10000 3000 10000 5300
 Wire Wire Line
-	6050 3000 10000 3000
+	6050 3000 8850 3000
 Wire Wire Line
 	8750 4400 9050 4400
@@
 Connection ~ 8850 3000
 Wire Wire Line
-	6050 5300 8950 5300
+	6050 5300 8850 5300
 Wire Wire Line
 	6050 4400 6050 5300
@@
 VCC
 $Comp
-L GND #PWR01
+L power:GND #PWR01
 U 1 1 59FCE2B5
 P 10600 3750
@@
 VCC
 $Comp
-L GND #PWR06
+L power:GND #PWR06
 U 1 1 59E63687
 P 8300 2250
@@
 $EndComp
 $Comp
-L PWR_FLAG #FLG02
+L power:PWR_FLAG #FLG02
 U 1 1 59FCE95A
 P 8300 2250
@@
 Wire Wire Line
 	10350 4000 10350 3750
+Wire Wire Line
+	8850 4200 9350 4200
+Wire Wire Line
+	8850 4300 9600 4300
+Wire Wire Line
+	9250 4000 9650 4000
+Wire Wire Line
+	8850 3000 10000 3000
+Wire Wire Line
+	8850 5300 8950 5300
 $EndSCHEMATC
